File: 0004-MCU-Datalogger.kicad_sch (KiCad schematic)
At the start: 25 parts, among them U1 24LC1025, U2 24LC1025, U3 DS1337S_, U4 ATMEGA328P-AU, Y1 Crystal, Y2 Crystal

Commit message: Assign values to components
Parts:
- C4: value C -> 0.1uF
- R5, R6: value R -> 10K
- Y2: value Crystal -> 32.768 KHz
Other:
- moved on the sheet: Y2
Changed lines of the file:
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@@
 			)
 		)
-		(property "Value" "R"
+		(property "Value" "10K"
 			(at 100.33 50.7999 0)
 			(effects
@@
 			)
 		)
-		(property "Value" "R"
+		(property "Value" "10K"
 			(at 111.76 50.7999 0)
 			(effects
@@
 	(symbol
 		(lib_id "Device:Crystal")
-		(at 27.94 62.23 0)
+		(at 29.21 59.69 90)
 		(unit 1)
 		(exclude_from_sim no)
@@
 		(fields_autoplaced yes)
 		(property "Reference" "Y2"
-			(at 27.94 54.61 0)
-			(effects
-				(font
-					(size 1.27 1.27)
-				)
-			)
-		)
-		(property "Value" "Crystal"
-			(at 27.94 57.15 0)
-			(effects
-				(font
-					(size 1.27 1.27)
-				)
-			)
-		)
-		(property "Footprint" ""
-			(at 27.94 62.23 0)
-			(effects
-				(font
-					(size 1.27 1.27)
-				)
-				(hide yes)
-			)
-		)
-		(property "Datasheet" "~"
-			(at 27.94 62.23 0)
+			(at 33.02 58.4199 90)
+			(effects
+				(font
+					(size 1.27 1.27)
+				)
+				(justify right)
+			)
+		)
+		(property "Value" "32.768 KHz"
+			(at 33.02 60.9599 90)
+			(effects
+				(font
+					(size 1.27 1.27)
+				)
+				(justify right)
+			)
+		)
+		(property "Footprint" ""
+			(at 29.21 59.69 0)
+			(effects
+				(font
+					(size 1.27 1.27)
+				)
+				(hide yes)
+			)
+		)
+		(property "Datasheet" "~"
+			(at 29.21 59.69 0)
 			(effects
 				(font
@@
 		)
 		(property "Description" "Two pin crystal"
-			(at 27.94 62.23 0)
-			(effects
-				(font
-					(size 1.27 1.27)
-				)
-				(hide yes)
+			(at 29.21 59.69 0)
+			(effects
+				(font
+					(size 1.27 1.27)
+				)
+				(hide yes)
+			)
+		)
+		(property "Purpose" ""
+			(at 29.21 59.69 0)
+			(effects
+				(font
+					(size 1.27 1.27)
+				)
 			)
 		)
@@
 			)
 		)
-		(property "Value" "C"
+		(property "Value" "0.1uF"
 			(at 123.19 50.7999 0)
 			(effects
@@
 			)
 		)
+		(property "Purpose" ""
+			(at 119.38 49.53 0)
+			(effects
+				(font
+					(size 1.27 1.27)
+				)
+			)
+		)

Commit message: Completed symbol footprint associations
Parts:
- BT1: footprint (none) -> Connector_PinHeader_2.54mm:PinHeader_1x02_P2.54mm_Vertical
- C1, C2: value C -> 22pF; footprint (none) -> Capacitor_SMD:C_0805_2012Metric
- C3: value C -> 0.1uF; footprint (none) -> Capacitor_SMD:C_0805_2012Metric
- C4: footprint (none) -> Capacitor_SMD:C_0805_2012Metric
- C5: value C_Polarized -> 100nF; footprint (none) -> Capacitor_SMD:C_0805_2012Metric
- D1, D2: footprint (none) -> LED_SMD:LED_0805_2012Metric
- H1, H2, H3, H4: footprint (none) -> MountingHole:MountingHole_2.1mm
- R1, R7: value R -> 330; footprint (none) -> Resistor_SMD:R_0805_2012Metric
- R2: value R -> 10K; footprint (none) -> Resistor_SMD:R_0805_2012Metric
- R3, R4: value R -> 4.7K; footprint (none) -> Resistor_SMD:R_0805_2012Metric
- R5, R6: footprint (none) -> Resistor_SMD:R_0805_2012Metric
- U1, U2: footprint (none) -> Package_SO:SOIC-8_5.23x5.23mm_P1.27mm
- Y1: value Crystal -> 16 MHz; footprint (none) -> Crystal:Crystal_SMD_5032-2Pin_5.0x3.2mm_HandSoldering
- Y2: footprint (none) -> Crystal:Crystal_SMD_5032-2Pin_5.0x3.2mm_HandSoldering
Other:
- moved on the sheet: R2, Y1
Changed lines of the file:
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@@
 			)
 		)
-		(property "Value" "R"
+		(property "Value" "330"
 			(at 241.3 81.2799 0)
 			(effects
@@
 			)
 		)
-		(property "Footprint" ""
+		(property "Footprint" "Resistor_SMD:R_0805_2012Metric"
 			(at 243.332 80.01 90)
 			(effects
@@
 			)
 		)
-		(property "Value" "R"
+		(property "Value" "4.7K"
 			(at 123.19 173.9899 0)
 			(effects
@@
 			)
 		)
-		(property "Footprint" ""
+		(property "Footprint" "Resistor_SMD:R_0805_2012Metric"
 			(at 118.872 172.72 90)
 			(effects
@@
 			)
 		)
-		(property "Footprint" ""
+		(property "Footprint" "Package_SO:SOIC-8_5.23x5.23mm_P1.27mm"
 			(at 58.42 171.45 0)
 			(effects
@@
 			)
 		)
-		(property "Value" "C"
+		(property "Value" "22pF"
 			(at 168.91 64.7699 0)
 			(effects
@@
 			)
 		)
-		(property "Footprint" ""
+		(property "Footprint" "Capacitor_SMD:C_0805_2012Metric"
 			(at 166.0652 67.31 0)
 			(effects
@@
 			)
 		)
-		(property "Value" "C"
+		(property "Value" "22pF"
 			(at 168.91 76.1999 0)
 			(effects
@@
 			)
 		)
-		(property "Footprint" ""
+		(property "Footprint" "Capacitor_SMD:C_0805_2012Metric"
 			(at 166.0652 78.74 0)
 			(effects
@@
 			)
 		)
-		(property "Footprint" ""
+		(property "Footprint" "Resistor_SMD:R_0805_2012Metric"
 			(at 96.012 49.53 90)
 			(effects
@@
 			)
 		)
-		(property "Footprint" ""
+		(property "Footprint" "MountingHole:MountingHole_2.1mm"
 			(at 241.3 142.24 0)
 			(effects
@@
 			)
 		)
-		(property "Footprint" ""
+		(property "Footprint" "MountingHole:MountingHole_2.1mm"
 			(at 241.3 152.4 0)
 			(effects
@@
 			)
 		)
-		(property "Value" "C_Polarized"
+		(property "Value" "100nF"
 			(at 250.19 43.5609 0)
 			(effects
@@
 			)
 		)
-		(property "Footprint" ""
+		(property "Footprint" "Capacitor_SMD:C_0805_2012Metric"
 			(at 247.3452 46.99 0)
 			(effects
@@
 			)
 		)
-		(property "Footprint" ""
+		(property "Footprint" "Resistor_SMD:R_0805_2012Metric"
 			(at 107.442 49.53 90)
 			(effects
@@
 			)
 		)
-		(property "Footprint" ""
+		(property "Footprint" "Crystal:Crystal_SMD_5032-2Pin_5.0x3.2mm_HandSoldering"
 			(at 29.21 59.69 0)
 			(effects
@@
 	(symbol
 		(lib_id "Device:Crystal")
-		(at 180.34 67.31 0)
+		(at 182.88 63.5 90)
 		(unit 1)
 		(exclude_from_sim no)
@@
 		(fields_autoplaced yes)
 		(property "Reference" "Y1"
-			(at 180.34 59.69 0)
-			(effects
-				(font
-					(size 1.27 1.27)
-				)
-			)
-		)
-		(property "Value" "Crystal"
-			(at 180.34 62.23 0)
-			(effects
-				(font
-					(size 1.27 1.27)
-				)
-			)
-		)
-		(property "Footprint" ""
-			(at 180.34 67.31 0)
+			(at 186.69 62.2299 90)
+			(effects
+				(font
+					(size 1.27 1.27)
+				)
+				(justify right)
+			)
+		)
+		(property "Value" "16 MHz"
+			(at 186.69 64.7699 90)
+			(effects
+				(font
+					(size 1.27 1.27)
+				)
+				(justify right)
+			)
+		)
+		(property "Footprint" "Crystal:Crystal_SMD_5032-2Pin_5.0x3.2mm_HandSoldering"
+			(at 182.88 63.5 0)
 			(effects
 				(font
@@
 		)
 		(property "Datasheet" "~"
-			(at 180.34 67.31 0)
+			(at 182.88 63.5 0)
 			(effects
 				(font
@@
 		)
 		(property "Description" "Two pin crystal"
-			(at 180.34 67.31 0)
+			(at 182.88 63.5 0)
 			(effects
 				(font
@@
 			)
 		)
-		(property "Footprint" ""
+		(property "Footprint" "Connector_PinHeader_2.54mm:PinHeader_1x02_P2.54mm_Vertical"
 			(at 264.16 41.656 90)
 			(effects
@@
 	(symbol
 		(lib_id "Device:R")
-		(at 36.83 149.86 0)
+		(at 184.15 86.36 90)
 		(unit 1)
 		(exclude_from_sim no)
@@
 		(fields_autoplaced yes)
 		(property "Reference" "R2"
-			(at 39.37 148.5899 0)
-			(effects
-				(font
-					(size 1.27 1.27)
-				)
-				(justify left)
-			)
-		)
-		(property "Value" "R"
-			(at 39.37 151.1299 0)
-			(effects
-				(font
-					(size 1.27 1.27)
-				)
-				(justify left)
-			)
-		)
-		(property "Footprint" ""
-			(at 35.052 149.86 90)
+			(at 184.15 80.01 90)
+			(effects
+				(font
+					(size 1.27 1.27)
+				)
+			)
+		)
+		(property "Value" "10K"
+			(at 184.15 82.55 90)
+			(effects
+				(font
+					(size 1.27 1.27)
+				)
+			)
+		)
+		(property "Footprint" "Resistor_SMD:R_0805_2012Metric"
+			(at 184.15 88.138 90)
 			(effects
 				(font
@@
 		)
 		(property "Datasheet" "~"
-			(at 36.83 149.86 0)
+			(at 184.15 86.36 0)
 			(effects
 				(font
@@
 		)
 		(property "Description" "Resistor"
-			(at 36.83 149.86 0)
+			(at 184.15 86.36 0)
 			(effects
 				(font
@@
 			)
 		)
-		(property "Footprint" ""
+		(property "Footprint" "Capacitor_SMD:C_0805_2012Metric"
 			(at 120.3452 53.34 0)
 			(effects
@@
 			)
 		)
-		(property "Value" "C"
+		(property "Value" "0.1uF"
 			(at 184.15 33.02 90)
 			(effects
@@
 			)
 		)
-		(property "Footprint" ""
+		(property "Footprint" "Capacitor_SMD:C_0805_2012Metric"
 			(at 187.96 37.1348 0)
 			(effects
@@
 			)
 		)
-		(property "Footprint" ""
+		(property "Footprint" "LED_SMD:LED_0805_2012Metric"
 			(at 185.42 50.8 0)
 			(effects
@@
 			)
 		)
-		(property "Value" "R"
+		(property "Value" "330"
 			(at 167.64 46.99 90)
 			(effects
@@
 			)
 		)
-		(property "Footprint" ""
+		(property "Footprint" "Resistor_SMD:R_0805_2012Metric"
 			(at 167.64 52.578 90)
 			(effects
@@
 			)
 		)
-		(property "Footprint" ""
+		(property "Footprint" "MountingHole:MountingHole_2.1mm"
 			(at 241.3 132.08 0)
 			(effects
@@
 			)
 		)
-		(property "Footprint" ""
+		(property "Footprint" "MountingHole:MountingHole_2.1mm"
 			(at 241.3 121.92 0)
 			(effects
@@
 			)
 		)
-		(property "Footprint" ""
+		(property "Footprint" "LED_SMD:LED_0805_2012Metric"
 			(at 242.57 63.5 0)
 			(effects
@@
 			)
 		)
-		(property "Footprint" ""
+		(property "Footprint" "Package_SO:SOIC-8_5.23x5.23mm_P1.27mm"
 			(at 95.25 172.72 0)
 			(effects
@@
 			)
 		)
-		(property "Value" "R"
+		(property "Value" "4.7K"
 			(at 135.89 173.9899 0)
 			(effects
@@
 			)
 		)
-		(property "Footprint" ""
+		(property "Footprint" "Resistor_SMD:R_0805_2012Metric"
 			(at 131.572 172.72 90)
 			(effects

Commit message: Complete wiring of main sheet
Parts:
- U3: footprint DS1337S_:SOIC127P600X175-8N -> Footprints:SOIC127P600X175-8N
- U4: footprint ATMEGA328P-AU:QFP80P900X900X120-32N -> Footprints:QFP80P900X900X120-32N
Connections:
- net at R1.1: now also D1.1 (K)
- net GND: now reaches R1.2
- net GND: now also C1.1, C2.1, C3.1, C4.2, R7.1, U1.4 (GND), U1.7 (WP), U2.2 (A1), U2.4 (GND), U2.7 (WP), U3.4 (GND), U4.21 (GND), U4.3 (GND), U4.5 (GND)
- net Vcc: now reaches R3.1
- net Vcc: now also C4.1, R2.1, R4.1, R5.1, R6.1, U1.1 (A0), U1.2 (A1), U1.3 (A2), U2.1 (A0), U2.3 (A2), U3.8 (VCC)
- net SCL: now reaches R3.2
- net SCL: now also D2.2 (A), U1.6 (SCL), U3.6 (SCL), U4.17 (PB5), U4.28 (PC5)
- net SDA: now reaches U1.5 (SDA)
- net SDA: now also R4.2, U3.5 (SDA), U4.27 (PC4)
- net at C2.2: now also U4.7 (PB6), Y1.2
- net at U3.1 (X1): now also Y2.2
- net at U3.2 (X2): now also Y2.1
- net at U3.3 (~{INTA}): now also R6.2
- net at U3.7 (SQW/~INT): now also R5.2
- net at C1.2: now also U4.8 (PB7), Y1.1
- net at C5.1: now also BT1.1 (+), D1.2 (A), U4.18 (AVCC), U4.4 (VCC)
- net RESET: now reaches R2.2
- net RESET: now also U4.29 (PC6/~{RESET})
- net D3: now reaches U4.1 (PD3)
- net D6: now reaches U4.10 (PD6)
- net D7: now reaches U4.11 (PD7)
- net D8: now reaches U4.12 (PB0)
- net MOSI: now reaches U4.15 (PB3)
- net MISO: now reaches U4.16 (PB4)
- net D4: now reaches U4.2 (PD4)
- net at U4.20 (AREF): now also C3.2
- net RX: now reaches U4.30 (PD0)
- net TX: now reaches U4.31 (PD1)
- net D2: now reaches U4.32 (PD2)
- net at U4.6 (VCC): no longer U4.4 (VCC)
- net D5: now reaches U4.9 (PD5)
- net at D2.1 (K): now also R7.2
- no-connect marks 0 -> 9
Other:
- moved on the sheet: BT1, C1, C2, C3, C4, C5, D1, D2, R1, R5, R6, R7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

Commit message: Complete wiring in the second sheet
Connections:
- net GND: now also BT1.2 (-), C5.2
- net SCL: now also U2.6 (SCL)
- net SDA: now also U2.5 (SDA)
- net Vcc: now also U1.8 (VCC), U2.8 (VCC)
Other:
- sheet Connectors ports: added D2, D3, D4, D5, D6, D7, D8, GND, MISO, MOSI, RESET, RX, SCL, SDA, TX, Vcc; removed none
