File: 0004-MCU-Datalogger.kicad_sch (KiCad schematic)
At the start: 25 parts, among them U1 24LC1025, U2 24LC1025, U3 DS1337S_, U4 ATMEGA328P-AU, Y1 16 MHz, Y2 32.768 KHz

Commit message: Completed comments
Other:
- note added: "EEPROM"
- note added: "MCU"
- note added: "Mounting"
- note added: "Real time clock"
- moved on the sheet: H1, H2, H3, H4

Commit message: Add Vcc Net Label to a battery circuit & Fix new routing violations
Connections:
- net Vcc: now also BT1.1 (+), C5.1, D1.2 (A), U4.18 (AVCC), U4.4 (VCC)
Changed lines of the file:
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@@
+		)
+	)
+	(label "Vcc"
+		(at 261.62 40.64 180)
+		(fields_autoplaced yes)
+		(effects
+			(font
+				(size 1.27 1.27)
+			)
+			(justify right bottom)
+		)
+		(property "Netclass" "Power"
+			(at 261.62 41.91 0)
+			(effects
+				(font
+					(size 1.27 1.27)
+					(italic yes)
+				)
+				(justify right)
+				(hide yes)
+			)
 		)
 	)

Commit message: Fix SCK issue
Connections:
- net SCL: no longer D2.2 (A), U4.17 (PB5)
- new net SCK: D2.2 (A), U4.17 (PB5)
Other:
- sheet Connectors ports: added SCK; removed none
Changed lines of the file:
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@@
 	)
 	(junction
+		(at 269.24 54.61)
+		(diameter 0)
+		(color 0 0 0 0)
+	)
+	(junction
 		(at 179.07 58.42)
 		(diameter 0)
@@
 	)
 	(junction
-		(at 269.24 55.245)
-		(diameter 0)
-		(color 0 0 0 0)
-	)
-	(junction
 		(at 243.84 81.28)
 		(diameter 0)
@@
 	(wire
 		(pts
-			(xy 83.82 46.99) (xy 86.995 46.99)
+			(xy 83.82 46.99) (xy 88.9 46.99)
 		)
 		(stroke
@@
 	(wire
 		(pts
-			(xy 86.995 46.99) (xy 86.995 39.37)
-		)
-		(stroke
-			(width 0)
-			(type default)
-		)
-	)
-	(wire
-		(pts
-			(xy 269.24 55.245) (xy 269.24 52.07)
+			(xy 88.9 46.99) (xy 88.9 39.37)
 		)
 		(stroke
@@
 	(wire
 		(pts
-			(xy 86.995 39.37) (xy 97.79 39.37)
+			(xy 88.9 39.37) (xy 97.79 39.37)
 		)
 		(stroke
@@
 	(wire
 		(pts
-			(xy 251.46 50.8) (xy 251.46 55.245)
+			(xy 251.46 50.8) (xy 251.46 54.61)
 		)
 		(stroke
@@
 	(wire
 		(pts
-			(xy 269.24 55.245) (xy 269.24 93.98)
+			(xy 269.24 54.61) (xy 269.24 93.98)
 		)
 		(stroke
@@
 	(wire
 		(pts
+			(xy 269.24 54.61) (xy 269.24 52.07)
+		)
+		(stroke
+			(width 0)
+			(type default)
+		)
+	)
+	(wire
+		(pts
 			(xy 88.9 69.85) (xy 88.9 74.93)
 		)
@@
 	(wire
 		(pts
-			(xy 251.46 55.245) (xy 269.24 55.245)
+			(xy 251.46 54.61) (xy 269.24 54.61)
 		)
 		(stroke
@@
 	(wire
 		(pts
-			(xy 243.84 35.56) (xy 243.84 40.64)
-		)
-		(stroke
-			(width 0)
-			(type default)
-		)
-	)
-	(wire
-		(pts
 			(xy 120.65 176.53) (xy 120.65 180.34)
 		)
@@
 	)
 	(label "MOSI"
-		(at 71.12 125.73 180)
+		(at 71.12 127 180)
 		(fields_autoplaced yes)
 		(effects
@@
 	)
 	(label "MISO"
-		(at 71.12 128.27 180)
+		(at 71.12 129.54 180)
 		(fields_autoplaced yes)
 		(effects
@@
 		)
 	)
-	(label "SCL"
+	(label "SCK"
 		(at 198.12 60.96 180)
 		(fields_autoplaced yes)
@@
 		)
 	)
+	(label "SCK"
+		(at 71.12 124.46 180)
+		(fields_autoplaced yes)
+		(effects
+			(font
+				(size 1.27 1.27)
+			)
+			(justify right bottom)
+		)
+	)
 	(label "RESET"
-		(at 71.12 130.81 180)
+		(at 71.12 132.08 180)
 		(fields_autoplaced yes)
 		(effects
@@
 	)
 	(symbol
-		(lib_id "power:PWR_FLAG")
-		(at 243.84 35.56 0)
-		(unit 1)
-		(exclude_from_sim no)
-		(in_bom yes)
-		(on_board yes)
-		(dnp no)
-		(fields_autoplaced yes)
-		(property "Reference" "#FLG01"
-			(at 243.84 33.655 0)
-			(effects
-				(font
-					(size 1.27 1.27)
-				)
-				(hide yes)
-			)
-		)
-		(property "Value" "PWR_FLAG"
-			(at 243.84 30.48 0)
-			(effects
-				(font
-					(size 1.27 1.27)
-				)
-			)
-		)
-		(property "Footprint" ""
-			(at 243.84 35.56 0)
-			(effects
-				(font
-					(size 1.27 1.27)
-				)
-				(hide yes)
-			)
-		)
-		(property "Datasheet" "~"
-			(at 243.84 35.56 0)
-			(effects
-				(font
-					(size 1.27 1.27)
-				)
-				(hide yes)
-			)
-		)
-		(property "Description" "Special symbol for telling ERC where power comes from"
-			(at 243.84 35.56 0)
-			(effects
-				(font
-					(size 1.27 1.27)
-				)
-				(hide yes)
-			)
-		)
-		(pin "1"
-		)
-		(instances
-			(project ""
-				(path "/8826d366-4ef5-455d-a76c-e91a1f47993d"
-					(reference "#FLG01")
-					(unit 1)
-				)
-			)
-		)
-	)
-	(symbol
 		(lib_id "Device:R")
 		(at 243.84 71.12 0)
@@
 		)
 		(pin "RESET" passive
-			(at 71.12 130.81 180)
+			(at 71.12 132.08 180)
 			(effects
 				(font
@@
 		)
 		(pin "MOSI" input
-			(at 71.12 125.73 180)
+			(at 71.12 127 180)
 			(effects
 				(font
@@
 		)
 		(pin "MISO" output
-			(at 71.12 128.27 180)
+			(at 71.12 129.54 180)
 			(effects
 				(font
@@
 			)
 		)
+		(pin "SCK" passive
+			(at 71.12 124.46 180)
+			(effects
+				(font
+					(size 1.27 1.27)
+				)
+				(justify left)
+			)
+		)
