File: 0004-MCU-Datalogger.kicad_pcb (KiCad board)
At the start: 2 copper layers, 29 parts, among them J1 Conn_01x04_Pin, J2 Conn_01x04_Pin, J3 Conn_01x09_Pin, J4 Conn_02x03_Odd_Even, U1 24LC1025, U2 24LC1025, U3 DS1337S_, U4 ATMEGA328P-AU, Y1 16 MHz, Y2 32.768 KHz

Commit message: Complete placement of footprints
Parts:
- moved H3 54.2 mm to (167.0, 62.2)
- moved R7 49.4 mm to (160.3, 61.6), turned to 180 degrees
- moved C5 46.4 mm to (150.5, 61.6), turned to 180 degrees
- moved H4 45.7 mm to (167.0, 85.7)
- moved C4 43.7 mm to (138.8, 61.6), turned to 180 degrees
- moved BT1 38.1 mm to (124.5, 67.9)
- moved D2 35.5 mm to (160.3, 64.8)
- moved R4 34.2 mm to (146.4, 61.6), turned to 180 degrees
- moved R1 34.1 mm to (156.2, 61.6), turned to 180 degrees
- moved C3 32.6 mm to (152.4, 69.8), turned to 180 degrees
- moved U3 31.7 mm to (132.0, 77.5)
- moved D1 31.6 mm to (156.2, 64.8), turned to 180 degrees
- moved U4 30.7 mm to (144.1, 69.8)
- moved J3 29.1 mm to (127.6, 85.7), turned to 90 degrees
- moved R3 27.8 mm to (152.4, 73.0), turned to 180 degrees
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Other:
- board outline added: 48.9 x 28.8 mm

Commit message: Finish routing
Parts:
- moved H1 0.63 mm to (123.2, 61.6)
- moved H3 0.63 mm to (167.0, 61.6)
- turned R2 to 0 degrees
Routing:
- net GND: track 0.00 -> 148.6 mm, vias 0 -> 9
- net /Vcc: track 0.00 -> 132.1 mm, vias 0 -> 4
- net /SCL: track 0.00 -> 72.3 mm, vias 0 -> 2
- net /SDA: track 0.00 -> 64.4 mm, vias 0 -> 2
- net Net-(BT1-+): track 0.00 -> 44.9 mm, vias 0 -> 3
- net /TX: track 0.00 -> 30.4 mm, vias 0 -> 1
- net /D2: track 0.00 -> 29.7 mm
- net /RX: track 0.00 -> 29.6 mm, vias 0 -> 1
- net /D3: track 0.00 -> 25.2 mm
- net /RESET: track 0.00 -> 24.1 mm, vias 0 -> 2
- net /D4: track 0.00 -> 22.3 mm
- net /MISO: track 0.00 -> 16.4 mm, vias 0 -> 2
- net Net-(U4-PB6): track 0.00 -> 15.9 mm, vias 0 -> 2
- net /D5: track 0.00 -> 14.8 mm
- net /MOSI: track 0.00 -> 14.3 mm
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Other:
- board size 48.9 x 28.8 mm -> 49.4 x 29.9 mm

Commit message: Finish edge cuts
Parts:
- moved H1 2.01 mm to (122.6, 59.7)
- moved H2 2.01 mm to (122.6, 87.6)
- moved H3 2.01 mm to (167.6, 59.7)
- moved H4 2.01 mm to (167.6, 87.6)
- moved J1 1.27 mm to (165.7, 69.8)
Routing:
- net /Vcc: track 132.1 -> 114.1 mm
- net /SDA: track 64.4 -> 63.1 mm
- net /SCL: track 72.3 -> 71.1 mm
Other:
- board size 49.4 x 29.9 mm -> 52.2 x 35.1 mm
Changed lines of the file:
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@@
 	(footprint "MountingHole:MountingHole_2.1mm"
 		(layer "F.Cu")
-		(at 167.005 61.595)
+		(at 167.64 59.69)
 		(descr "Mounting Hole 2.1mm, no annular")
 		(tags "mounting hole 2.1mm no annular")
@@
 	(footprint "Connector_PinHeader_2.54mm:PinHeader_1x04_P2.54mm_Vertical"
 		(layer "F.Cu")
-		(at 167.005 69.85)
+		(at 165.735 69.85)
 		(descr "Through hole straight pin header, 1x04, 2.54mm pitch, single row")
 		(tags "Through hole pin header THT 1x04 2.54mm single row")
@@
 	(footprint "MountingHole:MountingHole_2.1mm"
 		(layer "F.Cu")
-		(at 167.005 85.725)
+		(at 167.64 87.63)
 		(descr "Mounting Hole 2.1mm, no annular")
 		(tags "mounting hole 2.1mm no annular")
@@
 	(footprint "MountingHole:MountingHole_2.1mm"
 		(layer "F.Cu")
-		(at 123.19 85.725)
+		(at 122.555 87.63)
 		(descr "Mounting Hole 2.1mm, no annular")
 		(tags "mounting hole 2.1mm no annular")
@@
 	(footprint "MountingHole:MountingHole_2.1mm"
 		(layer "F.Cu")
-		(at 123.19 61.595)
+		(at 122.555 59.69)
 		(descr "Mounting Hole 2.1mm, no annular")
 		(tags "mounting hole 2.1mm no annular")
@@
 		)
 	)
-	(gr_line
-		(start 122.164987 83.03434)
-		(end 122.164987 64.262)
-		(stroke
-			(width 0.05)
-			(type default)
-		)
-		(layer "Edge.Cuts")
-	)
-	(gr_arc
-		(start 165.106776 59.704621)
-		(mid 168.830891 59.621835)
-		(end 169.050442 63.340394)
-		(stroke
-			(width 0.05)
-			(type default)
-		)
-		(layer "Edge.Cuts")
-	)
 	(gr_arc
-		(start 125.095 87.884)
-		(mid 120.725574 87.213929)
-		(end 122.164987 83.03434)
-		(stroke
-			(width 0.05)
-			(type default)
-		)
-		(layer "Edge.Cuts")
-	)
-	(gr_line
-		(start 169.050442 83.935238)
-		(end 169.050442 64.262)
+		(start 126.111 88.011)
+		(mid 120.070985 90.202929)
+		(end 122.049227 84.089592)
 		(stroke
 			(width 0.05)
@@
 	)
 	(gr_arc
-		(start 169.050442 83.935238)
-		(mid 168.989206 87.582419)
-		(end 165.354 87.883999)
+		(start 164.084 59.563)
+		(mid 170.06514 57.086164)
+		(end 168.019073 63.228017)
 		(stroke
 			(width 0.05)
@@
 	)
 	(gr_arc
-		(start 122.164987 64.262)
-		(mid 120.843816 59.964368)
-		(end 125.33243 59.704621)
+		(start 122.051785 63.212505)
+		(mid 120.176009 57.043933)
+		(end 126.111 59.563)
 		(stroke
 			(width 0.05)
@@
 	)
 	(gr_line
-		(start 165.1 87.884)
-		(end 125.095 87.884)
+		(start 122.049227 84.089592)
+		(end 122.052106 63.21026)
 		(stroke
 			(width 0.05)
@@
 	)
 	(gr_line
-		(start 125.33243 59.704621)
-		(end 165.1 59.704621)
+		(start 168.019073 63.228017)
+		(end 168.019073 84.095764)
 		(stroke
 			(width 0.05)
@@
 		(layer "Edge.Cuts")
 	)
-	(gr_line
-		(start 169.050442 64.262)
-		(end 169.050442 63.627)
+	(gr_arc
+		(start 168.021764 84.095764)
+		(mid 170.152531 90.144708)
+		(end 164.105435 88.008704)
 		(stroke
 			(width 0.05)
@@
 	)
 	(gr_line
-		(start 165.1 87.884)
-		(end 165.354 87.884)
+		(start 126.111 88.011)
+		(end 164.101983 88.009073)
 		(stroke
 			(width 0.05)
@@
 	)
 	(gr_line
-		(start 169.050442 63.627)
-		(end 169.050442 63.340394)
+		(start 126.111 59.563)
+		(end 164.084 59.563)
 		(stroke
 			(width 0.05)
@@
 	)
 	(segment
+		(start 165.862 66.294)
+		(end 161.21 61.642)
+		(width 0.35)
+		(layer "F.Cu")
+		(net 1)
+	)
+	(segment
 		(start 132.792672 71.54)
 		(end 135.332672 69)
@@
 	)
 	(segment
-		(start 167.005 67.39)
-		(end 161.21 61.595)
-		(width 0.35)
-		(layer "F.Cu")
-		(net 1)
-	)
-	(segment
 		(start 154.605 71.105)
 		(end 153.35 69.85)
@@
 	)
 	(segment
+		(start 165.862 69.85)
+		(end 165.862 66.294)
+		(width 0.35)
+		(layer "F.Cu")
+		(net 1)
+	)
+	(segment
 		(start 131.375 78.525)
 		(end 131.375 74.435)
@@
 	)
 	(segment
-		(start 167.005 69.85)
-		(end 167.005 67.39)
-		(width 0.35)
-		(layer "F.Cu")
-		(net 1)
-	)
-	(segment
 		(start 161.21 61.595)
 		(end 161.21 60.626)
@@
 	)
 	(segment
+		(start 161.21 61.642)
+		(end 161.21 61.595)
+		(width 0.35)
+		(layer "F.Cu")
+		(net 1)
+	)
+	(segment
 		(start 131.826 64.77)
 		(end 134.366 62.23)
@@
 	)
 	(segment
-		(start 168.28 73.665)
-		(end 168.28 77.998123)
-		(width 0.35)
-		(layer "F.Cu")
-		(net 6)
-	)
-	(segment
 		(start 149.24 84.45)
 		(end 154.935 84.45)
@@
 	)
 	(segment
-		(start 158.345 78.745)
-		(end 158.115 78.975)
-		(width 0.35)
-		(layer "F.Cu")
-		(net 6)
-	)
-	(segment
 		(start 146.152 60.452)
 		(end 142.803 60.452)
@@
 	)
 	(segment
-		(start 167.533123 78.745)
-		(end 158.345 78.745)
-		(width 0.35)
-		(layer "F.Cu")
-		(net 6)
-	)
-	(segment
 		(start 128.48 60.96)
 		(end 135.68 60.96)
@@
 	)
 	(segment
-		(start 168.28 77.998123)
-		(end 167.533123 78.745)
-		(width 0.35)
-		(layer "F.Cu")
-		(net 6)
-	)
-	(segment
 		(start 128.944 67.73)
 		(end 128.48 67.73)
@@
 	)
 	(segment
-		(start 167.005 72.39)
-		(end 168.28 73.665)
-		(width 0.35)
-		(layer "F.Cu")
-		(net 6)
-	)
-	(segment
 		(start 138.5625 60.445)
 		(end 139.7125 61.595)
@@
 	)
 	(segment
-		(start 161.925 67.31)
-		(end 155.229 67.31)
+		(start 155.229 67.31)
+		(end 160.655 67.31)
 		(width 0.35)
 		(layer "B.Cu")
@@
 	)
 	(segment
-		(start 167.005 72.39)
-		(end 161.925 67.31)
+		(start 155.448 74.422)
+		(end 156.352 74.422)
 		(width 0.35)
 		(layer "B.Cu")
@@
 	)
 	(segment
-		(start 155.448 74.422)
-		(end 156.352 74.422)
+		(start 160.655 67.31)
+		(end 165.735 72.39)
 		(width 0.35)
 		(layer "B.Cu")
@@
 	)
 	(segment
-		(start 155.229 67.31)
-		(end 155.194 67.275)
+		(start 155.194 67.275)
+		(end 155.229 67.31)
 		(width 0.35)
 		(layer "B.Cu")
@@
 	)
 	(segment
-		(start 163.18 73.645)
-		(end 167.005 77.47)
-		(width 0.25)
-		(layer "F.Cu")
-		(net 8)
-	)
-	(segment
 		(start 161.26 64.77)
 		(end 161.83 65.34)
@@
 	)
 	(segment
+		(start 161.91 73.645)
+		(end 165.735 77.47)
+		(width 0.25)
+		(layer "F.Cu")
+		(net 8)
+	)
+	(segment
 		(start 136.232 70.27)
 		(end 135.68 70.27)
@@
 	)
 	(segment
-		(start 160.655 73.645)
-		(end 163.18 73.645)
+		(start 134.366 72.898)
+		(end 134.366 70.866)
 		(width 0.25)
 		(layer "F.Cu")
@@
 	)
 	(segment
-		(start 134.366 72.898)
-		(end 134.366 70.866)
+		(start 160.655 73.645)
+		(end 161.91 73.645)
 		(width 0.25)
 		(layer "F.Cu")
@@
 	)
 	(segment
-		(start 164.525 77.41)
-		(end 167.005 74.93)
+		(start 152.0582 72.198927)
+		(end 157.269273 77.41)
 		(width 0.25)
 		(layer "B.Cu")
@@
 	)
 	(segment
-		(start 150.174105 64.262)
-		(end 152.0582 66.146095)
+		(start 157.269273 77.41)
+		(end 163.255 77.41)
 		(width 0.25)
 		(layer "B.Cu")
@@
 	)
 	(segment
-		(start 138.159 64.025)
-		(end 138.0744 64.1096)
+		(start 150.174105 64.262)
+		(end 152.0582 66.146095)
 		(width 0.25)
 		(layer "B.Cu")
@@
 	)
 	(segment
-		(start 145.542 64.025)
-		(end 138.159 64.025)
+		(start 163.255 77.41)
+		(end 165.735 74.93)
 		(width 0.25)
 		(layer "B.Cu")
@@
 	)
 	(segment
-		(start 150.174105 64.262)
-		(end 145.779 64.262)
+		(start 138.159 64.025)
+		(end 138.0744 64.1096)
 		(width 0.25)
 		(layer "B.Cu")
@@
 	)
 	(segment
-		(start 157.269273 77.41)
-		(end 164.525 77.41)
+		(start 145.542 64.025)
+		(end 138.159 64.025)
 		(width 0.25)
 		(layer "B.Cu")
@@
 	)
 	(segment
-		(start 145.779 64.262)
-		(end 145.542 64.025)
+		(start 152.0582 66.146095)
+		(end 152.0582 72.198927)
 		(width 0.25)
 		(layer "B.Cu")
@@
 	)
 	(segment
-		(start 152.0582 72.198927)
-		(end 157.269273 77.41)
+		(start 145.779 64.262)
+		(end 150.174105 64.262)
 		(width 0.25)
 		(layer "B.Cu")
@@
 	)
 	(segment
-		(start 152.0582 66.146095)
-		(end 152.0582 72.198927)
+		(start 145.542 64.025)
+		(end 145.779 64.262)
 		(width 0.25)
 		(layer "B.Cu")

Commit message: Add copper fills
Routing:
- net GND: track 148.2 -> 138.0 mm
- added copper zone on F.Cu, net /Vcc
- added copper zone on B.Cu, net GND
Changed lines of the file:
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@@
-	)
-	(segment
-		(start 165.862 66.294)
-		(end 161.21 61.642)
-		(width 0.35)
-		(layer "F.Cu")
-		(net 1)
 	)
 	(segment
@@
 	)
 	(segment
-		(start 165.862 69.85)
-		(end 165.862 66.294)
-		(width 0.35)
-		(layer "F.Cu")
-		(net 1)
-	)
-	(segment
 		(start 131.375 78.525)
 		(end 131.375 74.435)
@@
 		(net 26)
 	)
+	(zone
+		(net 6)
+		(net_name "/Vcc")
+		(layer "F.Cu")
+		(hatch edge 0.5)
+		(connect_pads
+			(clearance 0.5)
+		)
+		(min_thickness 0.25)
+		(filled_areas_thickness no)
+		(fill yes
+			(mode hatch)
+			(thermal_gap 0.5)
+			(thermal_bridge_width 0.5)
+			(hatch_thickness 1)
+			(hatch_gap 1.5)
+			(hatch_orientation 0)
+			(hatch_border_algorithm hatch_thickness)
+			(hatch_min_hole_area 0.3)
+		)
+		(polygon
+			(pts
+				(xy 163.9735 59.6735) (xy 125.8735 59.6735) (xy 122.1905 63.3565) (xy 122.1905 83.6765) (xy 126.3815 87.8675)
+				(xy 163.9735 87.8675) (xy 167.9105 83.9305) (xy 167.9105 63.6105)
+			)
+		)
+	)
+	(zone
+		(net 1)
+		(net_name "GND")
+		(layer "B.Cu")
+		(hatch edge 0.5)
+		(connect_pads
+			(clearance 0.5)
+		)
+		(min_thickness 0.25)
+		(filled_areas_thickness no)
+		(fill yes
+			(mode hatch)
+			(thermal_gap 0.5)
+			(thermal_bridge_width 0.5)
+			(hatch_thickness 1)
+			(hatch_gap 1.5)
+			(hatch_orientation 0)
+			(hatch_border_algorithm hatch_thickness)
+			(hatch_min_hole_area 0.3)
+		)
+		(polygon
+			(pts
+				(xy 163.957 59.69) (xy 125.857 59.69) (xy 122.174 63.373) (xy 122.174 83.693) (xy 126.365 87.884)
+				(xy 163.957 87.884) (xy 167.894 83.947) (xy 167.894 63.627)
+			)
+		)
+	)
 )

Commit message: Add Vcc Net Label to a battery circuit & Fix new routing violations
Parts:
- moved C1 0.63 mm to (141.6, 81.9)
- moved C2 0.63 mm to (146.7, 81.9)
- moved Y1 0.63 mm to (144.1, 78.1)
Connections:
- BT1 pad 1: Net-(BT1-+) -> /Vcc
- C5 pad 1: Net-(BT1-+) -> /Vcc
- D1 pad 2: Net-(BT1-+) -> /Vcc
- U4 pad 18: Net-(BT1-+) -> /Vcc
- U4 pad 4: Net-(BT1-+) -> /Vcc
Routing:
- net /Vcc: track 114.1 -> 159.3 mm, vias 4 -> 7
- net Net-(BT1-+): track 44.9 -> 0.00 mm, vias 3 -> 0
- net /SDA: track 63.1 -> 64.1 mm
Other:
- board text added: "1"
- board text added: "2"
- board text added: "3"
- board text added: "4"
- board text added: "5"
- board text added: "6"
- board text added: "7"
- board text added: "GND"
- board text added: "GND MOSI VCC"
- board text added: "RST SCL MISO"
- board text added: "RX"
- board text added: "SCL"
- board text added: "SDA"
- board text added: "TX"
- board text added: "VCC"

Commit message: Fix SCK issue
Parts:
- added REF**: KiCad-Logo2_5mm_SilkScreen, Symbol:KiCad-Logo2_5mm_SilkScreen, B.Cu at (158.6, 63.8)
Other:
- board text added: "Data logger with ATMega328P vbozic"

Commit message: Fix SCK issue in PCB editor
Connections:
- D2 pad 2: /SCL -> /SCK
- J4 pad 3: /SCL -> /SCK
- U4 pad 17: /SCL -> /SCK
Routing:
- net /SCK: track 0.00 -> 23.7 mm
- net /SCL: track 71.1 -> 63.1 mm, vias 2 -> 8
- net /Vcc: track 159.3 -> 160.5 mm
Changed lines of the file:
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@@
 	(net 33 "unconnected-(U4-PC1-Pad24)")
 	(net 34 "unconnected-(U4-ADC7-Pad22)")
+	(net 35 "/SCK")
 	(footprint "Resistor_SMD:R_0805_2012Metric"
 		(layer "F.Cu")
@@
 			(layers "F.Cu" "F.Paste" "F.Mask")
 			(roundrect_rratio 0.25)
-			(net 7 "/SCL")
+			(net 35 "/SCK")
 			(pinfunction "A")
 			(pintype "passive")
@@
 			(layers "*.Cu" "*.Mask")
 			(remove_unused_layers no)
-			(net 7 "/SCL")
+			(net 35 "/SCK")
 			(pinfunction "Pin_3")
 			(pintype "passive")
@@
 			(layers "F.Cu" "F.Paste" "F.Mask")
 			(roundrect_rratio 0.125)
-			(net 7 "/SCL")
+			(net 35 "/SCK")
 			(pinfunction "PB5")
 			(pintype "bidirectional")
@@
 	)
 	(segment
-		(start 158.115 78.975)
-		(end 158.115 83.82)
-		(width 0.35)
-		(layer "F.Cu")
-		(net 5)
-	)
-	(segment
 		(start 139.975 69.45)
 		(end 141.5546 69.45)
@@
 	)
 	(segment
+		(start 159.512 77.582)
+		(end 159.512 82.423)
+		(width 0.35)
+		(layer "F.Cu")
+		(net 5)
+	)
+	(segment
 		(start 134.49 75.565)
 		(end 133.505 75.565)
@@
 	)
 	(segment
+		(start 159.512 82.423)
+		(end 156.21 85.725)
+		(width 0.35)
+		(layer "F.Cu")
+		(net 5)
+	)
+	(segment
 		(start 128.944 67.73)
 		(end 128.48 67.73)
@@
 	)
 	(segment
-		(start 158.115 83.82)
-		(end 156.21 85.725)
-		(width 0.35)
-		(layer "F.Cu")
-		(net 5)
-	)
-	(segment
 		(start 128.48 63.5)
 		(end 128.48 62.23)
@@
 	)
 	(segment
-		(start 158.115 76.185)
-		(end 158.115 78.975)
-		(width 0.35)
-		(layer "F.Cu")
-		(net 5)
-	)
-	(segment
 		(start 135.68 60.96)
 		(end 136.195 60.445)
@@
 	)
 	(segment
+		(start 158.115 76.185)
+		(end 159.512 77.582)
+		(width 0.35)
+		(layer "F.Cu")
+		(net 5)
+	)
+	(segment
 		(start 139.7125 61.595)
 		(end 141.66 61.595)
@@
 	)
 	(segment
-		(start 144.545 65.68)
-		(end 144.545 66.311252)
+		(start 164.0586 79.1464)
+		(end 162.9156 79.1464)
 		(width 0.25)
 		(layer "F.Cu")
@@
 	)
 	(segment
-		(start 151.1125 72.65)
-		(end 151.4875 73.025)
+		(start 154.8246 79.1464)
+		(end 153.3652 77.687)
 		(width 0.25)
 		(layer "F.Cu")
@@
 	)
 	(segment
-		(start 147.574874 72.65)
-		(end 148.315 72.65)
+		(start 144.545 66.415)
+		(end 144.545 65.68)
 		(width 0.25)
 		(layer "F.Cu")
@@
 	)
 	(segment
-		(start 161.26 64.77)
-		(end 161.83 65.34)
+		(start 145.796 69.85)
+		(end 145.796 67.666)
 		(width 0.25)
 		(layer "F.Cu")
@@
 	)
 	(segment
-		(start 145.796 67.562252)
-		(end 145.796 70.871126)
+		(start 150.1394 73.025)
+		(end 150.0124 72.898)
 		(width 0.25)
 		(layer "F.Cu")
@@
 	)
 	(segment
-		(start 152.5625 71.95)
-		(end 156.786 71.95)
-		(width 0.25)
-		(layer "F.Cu")
-		(net 7)
-	)
-	(segment
-		(start 145.796 70.871126)
-		(end 147.574874 72.65)
+		(start 151.4875 73.025)
+		(end 150.1394 73.025)
 		(width 0.25)
 		(layer "F.Cu")
@@
 	)
 	(segment
-		(start 151.4875 73.025)
-		(end 152.5625 71.95)
+		(start 151.4875 75.171201)
+		(end 151.4875 73.025)
 		(width 0.25)
 		(layer "F.Cu")
@@
 	)
 	(segment
-		(start 161.83 65.34)
-		(end 161.83 72.47)
+		(start 158.3944 79.1464)
+		(end 154.8246 79.1464)
 		(width 0.25)
 		(layer "F.Cu")
@@
 	)
 	(segment
-		(start 156.786 71.95)
-		(end 157.306 72.47)
+		(start 165.735 77.47)
+		(end 164.0586 79.1464)
 		(width 0.25)
 		(layer "F.Cu")
@@
 	)
 	(segment
-		(start 144.545 66.311252)
-		(end 145.796 67.562252)
+		(start 146.558 70.612)
+		(end 145.796 69.85)
 		(width 0.25)
 		(layer "F.Cu")
@@
 	)
 	(segment
-		(start 134.880001 63.5)
-		(end 134.555 63.825001)
-		(width 0.25)
-		(layer "F.Cu")
-		(net 7)
-	)
-	(segment
-		(start 144.545 63.265)
-		(end 144.545 65.68)
+		(start 145.796 67.666)
+		(end 144.545 66.415)
 		(width 0.25)
 		(layer "F.Cu")
@@
 	)
 	(segment
-		(start 161.83 72.47)
-		(end 160.655 73.645)
+		(start 134.880001 63.5)
+		(end 134.555 63.825001)
 		(width 0.25)
 		(layer "F.Cu")
@@
 	)
 	(segment
-		(start 159.48 72.47)
-		(end 160.655 73.645)
+		(start 144.545 63.265)
+		(end 144.545 65.68)
 		(width 0.25)
 		(layer "F.Cu")
@@
 	)
 	(segment
-		(start 148.315 72.65)
-		(end 151.1125 72.65)
-		(width 0.25)
-		(layer "F.Cu")
-		(net 7)
-	)
-	(segment
 		(start 137.065 69.437)
 		(end 136.906 69.596)
@@
 	)
 	(segment
-		(start 157.306 72.47)
-		(end 159.48 72.47)
-		(width 0.25)
-		(layer "F.Cu")
-		(net 7)
-	)
-	(segment
 		(start 135.475 78.105)
 		(end 136.144 77.436)
@@
 	)
 	(segment
-		(start 161.91 73.645)
-		(end 165.735 77.47)
-		(width 0.25)
-		(layer "F.Cu")
-		(net 7)
-	)
-	(segment
 		(start 136.232 70.27)
 		(end 135.68 70.27)
@@
 	)
 	(segment
-		(start 134.366 72.898)
-		(end 134.366 70.866)
+		(start 151.7913 75.475001)
+		(end 151.4875 75.171201)
 		(width 0.25)
 		(layer "F.Cu")
@@
 	)
 	(segment
-		(start 160.655 73.645)
-		(end 161.91 73.645)
+		(start 134.366 72.898)
+		(end 134.366 70.866)
 		(width 0.25)
 		(layer "F.Cu")
@@
 	)
 	(via
+		(at 158.3944 79.1464)
+		(size 0.8)
+		(drill 0.4)
+		(layers "F.Cu" "B.Cu")
+		(net 7)
+	)
+	(via
+		(at 150.0124 72.898)
+		(size 0.8)
+		(drill 0.4)
+		(layers "F.Cu" "B.Cu")
+		(net 7)
+	)
+	(via
+		(at 151.7913 75.475001)
+		(size 0.8)
+		(drill 0.4)
+		(layers "F.Cu" "B.Cu")
+		(net 7)
+	)
+	(via
+		(at 153.3652 77.687)
+		(size 0.8)
+		(drill 0.4)
+		(layers "F.Cu" "B.Cu")
+		(net 7)
+	)
+	(via
+		(at 162.9156 79.1464)
+		(size 0.8)
+		(drill 0.4)
+		(layers "F.Cu" "B.Cu")
+		(net 7)
+	)
+	(via
 		(at 139.0904 63.246)
 		(size 0.8)
@@
 		(net 7)
 	)
+	(via
+		(at 146.558 70.612)
+		(size 0.8)
+		(drill 0.4)
+		(layers "F.Cu" "B.Cu")
+		(net 7)
+	)
+	(segment
+		(start 153.162 77.4838)
+		(end 153.162 76.845701)
+		(width 0.25)
+		(layer "B.Cu")
+		(net 7)
+	)
+	(segment
+		(start 149.606 72.898)
+		(end 147.32 70.612)
+		(width 0.25)
+		(layer "B.Cu")
+		(net 7)
+	)
 	(segment
 		(start 144.526 63.246)
@@
 	)
 	(segment
+		(start 162.9156 79.1464)
+		(end 158.3944 79.1464)
+		(width 0.25)
+		(layer "B.Cu")
+		(net 7)
+	)
+	(segment
+		(start 147.32 70.612)
+		(end 146.558 70.612)
+		(width 0.25)
+		(layer "B.Cu")
+		(net 7)
+	)
+	(segment
+		(start 150.0124 72.898)
+		(end 149.606 72.898)
+		(width 0.25)
+		(layer "B.Cu")
+		(net 7)
+	)
+	(segment
 		(start 139.446 63.246)
 		(end 139.0904 63.246)
@@
 	)
 	(segment
+		(start 153.3652 77.687)
+		(end 153.162 77.4838)
+		(width 0.25)
+		(layer "B.Cu")
+		(net 7)
+	)
+	(segment
+		(start 153.162 76.845701)
+		(end 151.7913 75.475001)
+		(width 0.25)
+		(layer "B.Cu")
+		(net 7)
+	)
+	(segment
 		(start 159.385 61.595)
 		(end 159.385 64.77)
@@
 		(net 25)
 	)
+	(segment
+		(start 160.655 73.645)
+		(end 159.48 72.47)
+		(width 0.25)
+		(layer "F.Cu")
+		(net 35)
+	)
+	(segment
+		(start 147.574874 72.65)
+		(end 148.315 72.65)
+		(width 0.25)
+		(layer "F.Cu")
+		(net 35)
+	)
+	(segment
+		(start 157.306 72.47)
+		(end 156.786 71.95)
+		(width 0.25)
+		(layer "F.Cu")
+		(net 35)
+	)
+	(segment
+		(start 159.48 72.47)
+		(end 157.306 72.47)
+		(width 0.25)
+		(layer "F.Cu")
+		(net 35)
+	)
+	(segment
+		(start 156.786 71.95)
+		(end 149.795306 71.95)
+		(width 0.25)
+		(layer "F.Cu")
+		(net 35)
+	)
+	(segment
+		(start 161.26 64.77)
+		(end 161.83 65.34)
+		(width 0.25)
+		(layer "F.Cu")
+		(net 35)
+	)
+	(segment
+		(start 161.83 65.34)
+		(end 161.83 72.47)
+		(width 0.25)
+		(layer "F.Cu")
+		(net 35)
+	)
+	(segment
+		(start 149.795306 71.95)
+		(end 149.095306 72.65)
+		(width 0.25)
+		(layer "F.Cu")
+		(net 35)
+	)
+	(segment
+		(start 161.83 72.47)
+		(end 160.655 73.645)
+		(width 0.25)
+		(layer "F.Cu")
+		(net 35)
+	)
+	(segment
+		(start 149.095306 72.65)
+		(end 148.315 72.65)
+		(width 0.25)
+		(layer "F.Cu")
+		(net 35)
+	)
 	(zone
